File: KiCAD/KZ80-YM2149.sch (KiCad schematic (older format))
At the start: 27 parts, among them J1 ADDR JP, J2 Conn_01x02, J3 SBC8080 BUS, U1 74HC00, U2 74HC138, U3 74HC02, U4 74HC74, U5 YM2149, Y1 3.57MHz

Commit message: ジョイスティックポート接続&プリントパターン見直し
Parts:
- removed J2: Conn_01x02, Connector_PinHeader_2.54mm:PinHeader_1x02_P2.54mm_Horizontal, symbol Connector_Generic:Conn_01x02
- added C1, C2: 1u, Capacitor_THT:CP_Radial_D5.0mm_P2.50mm, symbol Device:CP
- added C10, C11: 0.1u, Capacitor_THT:C_Disc_D3.0mm_W1.6mm_P2.50mm, symbol Device:C
- added J1: Audio-Jack-3_2Switches, AJ-1780:AJ-1780, symbol YM2151-rescue:Audio-Jack-3_2Switches
- added J3: JOYSTICK1, DSUB:DSUB-9_Male_Horizontal_P2.77x2.54mm_EdgePinOffset9.40mm, symbol Connector:DB9_Male_MountingHoles
- added J5: JOYSTICK2, DSUB:DSUB-9_Male_Horizontal_P2.77x2.54mm_EdgePinOffset9.40mm, symbol Connector:DB9_Male_MountingHoles
- added R3, R5: 2.2k, Resistor_THT:R_Axial_DIN0207_L6.3mm_D2.5mm_P10.16mm_Horizontal, symbol Device:R_US
- added RN1, RN2: 10k, Resistor_THT:R_Array_SIP9, symbol Device:R_Network08_US
- added U4, U7: 74HC157, Package_DIP:DIP-16_W7.62mm_Socket, symbol 74xx:74LS157
- R2: renamed from R4; value 1k -> 2.2k
- R6: value 2k -> 2.2k
- renumbered C8 to C12, C1 to C3, C2 to C4, C3 to C5, C4 to C6, C5 to C7, C6 to C8, C7 to C9, J1 to J2, J3 to J4, R3 to R1, R5 to R4, R1 to R7, R2 to R8, U2 to U1, U1 to U2, U4 to U5, U5 to U6
Connections:
- wire segments 195 -> 361
- no-connect marks 43 -> 42
Other:
- moved on the sheet: C12, C3, C4, C5, C6, C7, C8, C9, J2, J4, R1, R2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

Commit message: 回路図 クロック等 微修正
Parts:
- Y1: value 3.57MHz -> 3.579545MHz
Changed lines of the file:
@@
 P 2900 6050
 F 0 "Y1" H 3050 6100 50  0000 C CNN
-F 1 "3.57MHz" H 2950 5900 50  0000 C CNN
+F 1 "3.579545MHz" H 2950 5900 50  0000 C CNN
 F 2 "Crystal:Crystal_HC49-U_Vertical" H 2900 6050 50  0001 C CNN
 F 3 "~" H 2900 6050 50  0001 C CNN
@@
 U 1 1 5D08E7BD
 P 2500 6300
-F 0 "C3" H 2615 6346 50  0000 L CNN
-F 1 "22p" H 2615 6255 50  0000 L CNN
+F 0 "C3" H 2600 6300 50  0000 L CNN
+F 1 "22p" H 2600 6200 50  0000 L CNN
 F 2 "Capacitor_THT:C_Disc_D3.0mm_W1.6mm_P2.50mm" H 2538 6150 50  0001 C CNN
 F 3 "~" H 2500 6300 50  0001 C CNN
@@
 U 1 1 5D08E858
 P 3300 6300
-F 0 "C4" H 3415 6346 50  0000 L CNN
-F 1 "22p" H 3415 6255 50  0000 L CNN
+F 0 "C4" H 3400 6300 50  0000 L CNN
+F 1 "22p" H 3400 6200 50  0000 L CNN
 F 2 "Capacitor_THT:C_Disc_D3.0mm_W1.6mm_P2.50mm" H 3338 6150 50  0001 C CNN
 F 3 "~" H 3300 6300 50  0001 C CNN
