File: KiCAD/KZ80-YM2149.kicad_sch (KiCad schematic)
At the start: 55 parts

Commit message: コンデンサシンボル変更忘れ対応 #2
Parts:
- removed C1, C12, C2: (no value), symbol KZ80-YM2149-rescue:CP-Device
- added C1, C12: (no value), symbol Device:C_Polarized
- added C2: 1u, symbol Device:C_Polarized
- C10, C11, C13, C14, C5, C6, C7, C8, C9: value (none) -> 0.1u; footprint (none) -> Capacitor_THT:C_Disc_D3.0mm_W1.6mm_P2.50mm
- C3, C4: value (none) -> 22p; footprint (none) -> Capacitor_THT:C_Disc_D3.0mm_W1.6mm_P2.50mm
- D1: value (none) -> 1N4148; footprint (none) -> Diode_THT:D_DO-35_SOD27_P7.62mm_Horizontal
- J1: value (none) -> Audio-Jack-3_2Switches; footprint (none) -> AJ-1780:AJ-1780
- J2: value (none) -> ADDR JP; footprint (none) -> Connector_PinHeader_2.54mm:PinHeader_2x08_P2.54mm_Vertical
- J3: value (none) -> JOYSTICK1; footprint (none) -> DSUB:DSUB-9_Male_Horizontal_P2.77x2.54mm_EdgePinOffset9.40mm
- J4: value (none) -> SBC8080 BUS; footprint (none) -> Connector_PinHeader_2.54mm:PinHeader_2x20_P2.54mm_Horizontal
- J5: value (none) -> JOYSTICK2; footprint (none) -> DSUB:DSUB-9_Male_Horizontal_P2.77x2.54mm_EdgePinOffset9.40mm
- J6: value (none) -> CMT IN; footprint (none) -> AJ-1780:AJ-1780
- J7: value (none) -> SOUND-IN; footprint (none) -> Connector_PinHeader_2.54mm:PinHeader_1x02_P2.54mm_Vertical
- MH1, MH2, MH3, MH4, MH5, MH6: value (none) -> MountingHole; footprint (none) -> MountingHole:MountingHole_3.2mm_M3
- R1, R4, R8: value (none) -> 1k; footprint (none) -> Resistor_THT:R_Axial_DIN0207_L6.3mm_D2.5mm_P10.16mm_Horizontal
- R10: value (none) -> 470k; footprint (none) -> Resistor_THT:R_Axial_DIN0207_L6.3mm_D2.5mm_P10.16mm_Horizontal
- R11: value (none) -> 4.7k; footprint (none) -> Resistor_THT:R_Axial_DIN0207_L6.3mm_D2.5mm_P10.16mm_Horizontal
- R12: value (none) -> 12k; footprint (none) -> Resistor_THT:R_Axial_DIN0207_L6.3mm_D2.5mm_P10.16mm_Horizontal
- R13, R14, R15, R2, R3, R5, R6, R9: value (none) -> 2.2k; footprint (none) -> Resistor_THT:R_Axial_DIN0207_L6.3mm_D2.5mm_P10.16mm_Horizontal
- R7: value (none) -> 1M; footprint (none) -> Resistor_THT:R_Axial_DIN0207_L6.3mm_D2.5mm_P10.16mm_Horizontal
- RN1, RN2: value (none) -> 10k; footprint (none) -> Resistor_THT:R_Array_SIP9
- U1: value (none) -> 74HC138; footprint (none) -> Package_DIP:DIP-16_W7.62mm_Socket
- U2: value (none) -> 74HC00; footprint (none) -> Package_DIP:DIP-14_W7.62mm_Socket
- U3: value (none) -> 74HC02; footprint (none) -> Package_DIP:DIP-14_W7.62mm_Socket
- U4, U7: value (none) -> 74HC157; footprint (none) -> Package_DIP:DIP-16_W7.62mm_Socket
- U5: value (none) -> 74HC74; footprint (none) -> Package_DIP:DIP-14_W7.62mm_Socket
- U6: value (none) -> YM2149; footprint (none) -> Package_DIP:DIP-40_W15.24mm_Socket
- U8: value (none) -> LM311; footprint (none) -> Package_DIP:DIP-8_W7.62mm_Socket_LongPads
- Y1: value (none) -> 3.579545MHz; footprint (none) -> Crystal:Crystal_HC49-U_Vertical
Connections:
- net GND: now also C12.2
- net VCC: now also C12.1
- net at R1.1, R14.1, R2.1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: now also C1.1
- net at R15.1, R3.1, R4.1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: now also C2.1
- net at J1.2: now also C1.2
- net at J1.5: now also C2.2
